Commit message: Deleted Unneccesary

File: urdf/spider.xacro (robot description, xacro)
@@ -154,3 +154,45 @@
     </plugin>
   </gazebo>
+  <link name="imu_link">
+    <visual>
+      <origin xyz="0 0 0" rpy="0 0 0"/>
+      <geometry><box size="0.01 0.01 0.01"/></geometry>
+      <material name="grey"/>
+    </visual>
+    <inertial>
+      <mass value="0.01"/>
+      <inertia ixx="1e-5" ixy="0" ixz="0" iyy="1e-5" iyz="0" izz="1e-5"/>
+    </inertial>
+  </link>
+  <joint name="imu_joint" type="fixed">
+    <parent link="base_link"/>
+    <child link="imu_link"/>
+    <origin xyz="0 0 0.01" rpy="0 0 0"/>
+  </joint>
+  <gazebo reference="imu_link">
+    <sensor name="imu" type="imu">
+      <always_on>1</always_on>
+      <update_rate>50</update_rate>
+      <visualize>true</visualize>
+      <topic>imu/data</topic>
+      <enable_metrics>true</enable_metrics>
+      <ignition_frame_id>imu_link</ignition_frame_id>
+      <!-- <imu>
+        <angular_velocity>
+          <x><noise type="gaussian"><mean>0.0</mean><stddev>2e-4</stddev></noise></x>
+          <y><noise type="gaussian"><mean>0.0</mean><stddev>2e-4</stddev></noise></y>
+          <z><noise type="gaussian"><mean>0.0</mean><stddev>2e-4</stddev></noise></z>
+        </angular_velocity>
+        <linear_acceleration>
+          <x><noise type="gaussian"><mean>0.0</mean><stddev>1.7e-2</stddev></noise></x>
+          <y><noise type="gaussian"><mean>0.0</mean><stddev>1.7e-2</stddev></noise></y>
+          <z><noise type="gaussian"><mean>0.0</mean><stddev>1.7e-2</stddev></noise></z>
+        </linear_acceleration>
+      </imu> -->
+    </sensor>
+  </gazebo>
+  <gazebo>
+    <!-- <plugin filename="gz-sim-imu-system" name="gz::sim::systems::Imu"> -->
+    <plugin filename="libignition-gazebo-imu-system" name="ignition::gazebo::systems::Imu"/>
+  </gazebo>
 </robot>

Commit message: Lidar Added

File: urdf/spider.xacro (robot description, xacro)
@@ -196,3 +196,60 @@
     <plugin filename="libignition-gazebo-imu-system" name="ignition::gazebo::systems::Imu"/>
   </gazebo>
+  <link name="lidar_link">
+      <visual>
+          <origin xyz="0 0 0" rpy="0 0 3.1415"/>
+          <geometry>
+              <cylinder radius="0.02" length="0.02"/>
+          </geometry>
+      </visual>
+      <collision>
+          <origin xyz="0 0 0" rpy="-1.57 0 3.1415"/>
+          <geometry>
+              <cylinder radius="0.02" length="0.02"/>
+          </geometry>
+      </collision>
+        <self_collide>false</self_collide>
+  </link>
+  <joint name="lidar_to_payload" type="fixed">
+      <parent link="base_link"/>
+      <child link="lidar_link"/>
+      <origin xyz="0 0 0.065" rpy="0 0 3.1415"/>
+  </joint>
+  <gazebo reference="lidar_link">
+      <sensor name='gpu_lidar' type='gpu_lidar'>
+          <pose>0 0 0 0 0 0</pose>
+          <topic>scan</topic>
+          <frame_name>lidar_link</frame_name>
+          <gz_frame_id>lidar_link</gz_frame_id>
+          <update_rate>2</update_rate>
+          <lidar>
+              <scan>
+              <horizontal>
+                  <samples>720</samples>
+                  <resolution>1</resolution>
+                  <min_angle>-3.14159</min_angle>
+                  <max_angle>3.14159</max_angle>
+              </horizontal>
+              <vertical>
+                  <samples>1</samples>
+                  <resolution>1</resolution>
+                  <min_angle>0.0</min_angle>
+                  <max_angle>0.0</max_angle>
+              </vertical>
+              </scan>
+              <range>
+                  <min>0.01</min>
+                  <max>12.0</max>
+                  <resolution>0.005</resolution>
+              </range>
+              <noise>
+                  <type>gaussian</type>
+                  <mean>0.0</mean>
+                  <stddev>0.001</stddev>
+              </noise>
+          </lidar>
+          <always_on>true</always_on>
+          <visualize>true</visualize>
+      </sensor>
+  </gazebo>
 </robot>
